File: dclink.kicad_pcb (KiCad board)
At the start: 2 copper layers, 61.5 x 53.6 mm, 4 parts

Commit message: review
Other:
- board size 61.5 x 53.6 mm -> 61.5 x 52.6 mm
Changed lines of the file:
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@@
     (fp_rect (start -28.75 -7.75) (end 28.75 26.75) (layer "F.SilkS") (width 0.12) (fill none))
     (fp_rect (start 26.25 19.5) (end -26.25 -0.5) (layer "F.SilkS") (width 0.12) (fill none))
-    (pad "1" thru_hole circle (at -26.25 -0.5 180) (size 3 3) (drill 1.5) (layers *.Cu *.Mask)
+    (pad "1" thru_hole circle (at -26.25 -0.5 180) (size 4 4) (drill 1.8) (layers *.Cu *.Mask)
       (net 2 "VDC") (pinfunction "GND") (pintype "output") (zone_connect 2))
-    (pad "2" thru_hole circle (at 26.25 -0.5 180) (size 3 3) (drill 1.5) (layers *.Cu *.Mask)
+    (pad "2" thru_hole circle (at 26.25 -0.5 180) (size 4 4) (drill 1.8) (layers *.Cu *.Mask)
       (net 1 "GND") (pinfunction "GND") (pintype "output") (zone_connect 2))
-    (pad "3" thru_hole circle (at -26.25 19.5 180) (size 3 3) (drill 1.5) (layers *.Cu *.Mask)
+    (pad "3" thru_hole circle (at -26.25 19.5 180) (size 4 4) (drill 1.8) (layers *.Cu *.Mask)
       (net 2 "VDC") (pinfunction "SUP") (pintype "input") (zone_connect 2))
-    (pad "4" thru_hole circle (at 26.25 19.5 180) (size 3 3) (drill 1.5) (layers *.Cu *.Mask)
+    (pad "4" thru_hole circle (at 26.25 19.5 180) (size 4 4) (drill 1.8) (layers *.Cu *.Mask)
       (net 1 "GND") (pinfunction "GND") (pintype "output") (zone_connect 2))
   )
@@
       ) (layer "B.SilkS") (width 0) (fill solid))
   )
-  (gr_line (start 176.6 77.5) (end 164.6 77.5) (layer "F.Cu") (width 0.2))
-  (gr_line (start 123.1 77.5) (end 135.1 77.5) (layer "F.Cu") (width 0.2))
-  (gr_arc (start 176.6 77.5) (mid 179.428427 78.671573) (end 180.6 81.5) (layer "F.Cu") (width 0.2))
+  (gr_line (start 176.6 78.5) (end 164.6 78.5) (layer "F.Cu") (width 0.2))
+  (gr_line (start 123.1 78.5) (end 135.1 78.5) (layer "F.Cu") (width 0.2))
+  (gr_arc (start 176.6 78.5) (mid 179.428427 79.671573) (end 180.6 82.5) (layer "F.Cu") (width 0.2))
   (gr_arc (start 143.1 94.5) (mid 140.271573 93.328427) (end 139.1 90.5) (layer "F.Cu") (width 0.2))
-  (gr_line (start 160.6 81.5) (end 160.6 90.5) (layer "F.Cu") (width 0.2))
+  (gr_line (start 160.6 82.5) (end 160.6 90.5) (layer "F.Cu") (width 0.2))
   (gr_arc (start 160.6 90.5) (mid 159.428427 93.328427) (end 156.6 94.5) (layer "F.Cu") (width 0.2))
-  (gr_line (start 119.1 81.5) (end 119.1 127.1) (layer "F.Cu") (width 0.2))
-  (gr_line (start 180.6 94.2) (end 180.6 81.5) (layer "F.Cu") (width 0.2))
+  (gr_line (start 119.1 82.5) (end 119.1 127.1) (layer "F.Cu") (width 0.2))
+  (gr_line (start 180.6 94.2) (end 180.6 82.5) (layer "F.Cu") (width 0.2))
   (gr_arc (start 123.1 131.1) (mid 120.271573 129.928427) (end 119.1 127.1) (layer "F.Cu") (width 0.2))
-  (gr_arc (start 135.1 77.5) (mid 137.928427 78.671573) (end 139.1 81.5) (layer "F.Cu") (width 0.2))
-  (gr_arc (start 119.1 81.5) (mid 120.271573 78.671573) (end 123.1 77.5) (layer "F.Cu") (width 0.2))
+  (gr_arc (start 135.1 78.5) (mid 137.928427 79.671573) (end 139.1 82.5) (layer "F.Cu") (width 0.2))
+  (gr_arc (start 119.1 82.5) (mid 120.271573 79.671573) (end 123.1 78.5) (layer "F.Cu") (width 0.2))
   (gr_line (start 180.6 127.1) (end 180.6 94.2) (layer "F.Cu") (width 0.2))
-  (gr_arc (start 160.6 81.5) (mid 161.771573 78.671573) (end 164.6 77.5) (layer "F.Cu") (width 0.2))
+  (gr_arc (start 160.6 82.5) (mid 161.771573 79.671573) (end 164.6 78.5) (layer "F.Cu") (width 0.2))
   (gr_arc (start 180.6 127.1) (mid 179.428427 129.928427) (end 176.6 131.1) (layer "F.Cu") (width 0.2))
-  (gr_line (start 139.1 81.5) (end 139.1 90.5) (layer "F.Cu") (width 0.2))
+  (gr_line (start 139.1 82.5) (end 139.1 90.5) (layer "F.Cu") (width 0.2))
   (gr_line (start 156.6 94.5) (end 143.1 94.5) (layer "F.Cu") (width 0.2))
   (gr_line (start 123.1 131.1) (end 176.6 131.1) (layer "F.Cu") (width 0.2))
-  (gr_line (start 135.1 77.5) (end 123.1 77.5) (layer "Edge.Cuts") (width 0.05))
+  (gr_line (start 135.1 78.5) (end 123.1 78.5) (layer "Edge.Cuts") (width 0.05))
   (gr_line (start 123.1 131.1) (end 176.6 131.1) (layer "Edge.Cuts") (width 0.05))
-  (gr_line (start 160.6 81.5) (end 160.6 90.5) (layer "Edge.Cuts") (width 0.05))
-  (gr_line (start 139.1 90.5) (end 139.1 81.5) (layer "Edge.Cuts") (width 0.05))
-  (gr_arc (start 160.6 81.5) (mid 161.771573 78.671573) (end 164.6 77.5) (layer "Edge.Cuts") (width 0.05))
+  (gr_line (start 160.6 82.5) (end 160.6 90.5) (layer "Edge.Cuts") (width 0.05))
+  (gr_line (start 139.1 90.5) (end 139.1 82.5) (layer "Edge.Cuts") (width 0.05))
+  (gr_arc (start 160.6 82.5) (mid 161.771573 79.671573) (end 164.6 78.5) (layer "Edge.Cuts") (width 0.05))
   (gr_line (start 156.6 94.5) (end 143.1 94.5) (layer "Edge.Cuts") (width 0.05))
-  (gr_arc (start 176.6 77.5) (mid 179.428427 78.671573) (end 180.6 81.5) (layer "Edge.Cuts") (width 0.05))
+  (gr_arc (start 176.6 78.5) (mid 179.428427 79.671573) (end 180.6 82.5) (layer "Edge.Cuts") (width 0.05))
   (gr_arc (start 160.6 90.5) (mid 159.428427 93.328427) (end 156.6 94.5) (layer "Edge.Cuts") (width 0.05))
   (gr_arc (start 180.6 127.1) (mid 179.428427 129.928427) (end 176.6 131.1) (layer "Edge.Cuts") (width 0.05))
-  (gr_arc (start 119.1 81.5) (mid 120.271573 78.671573) (end 123.1 77.5) (layer "Edge.Cuts") (width 0.05))
+  (gr_arc (start 119.1 82.5) (mid 120.271573 79.671573) (end 123.1 78.5) (layer "Edge.Cuts") (width 0.05))
   (gr_arc (start 143.1 94.5) (mid 140.271573 93.328427) (end 139.1 90.5) (layer "Edge.Cuts") (width 0.05))
-  (gr_line (start 180.6 127.1) (end 180.6 81.5) (layer "Edge.Cuts") (width 0.05))
-  (gr_line (start 119.1 81.5) (end 119.1 127.1) (layer "Edge.Cuts") (width 0.05))
+  (gr_line (start 180.6 127.1) (end 180.6 82.5) (layer "Edge.Cuts") (width 0.05))
+  (gr_line (start 119.1 82.5) (end 119.1 127.1) (layer "Edge.Cuts") (width 0.05))
   (gr_arc (start 123.1 131.1) (mid 120.271573 129.928427) (end 119.1 127.1) (layer "Edge.Cuts") (width 0.05))
-  (gr_line (start 176.6 77.5) (end 164.6 77.5) (layer "Edge.Cuts") (width 0.05))
-  (gr_arc (start 135.1 77.5) (mid 137.928427 78.671573) (end 139.1 81.5) (layer "Edge.Cuts") (width 0.05))
+  (gr_line (start 176.6 78.5) (end 164.6 78.5) (layer "Edge.Cuts") (width 0.05))
+  (gr_arc (start 135.1 78.5) (mid 137.928427 79.671573) (end 139.1 82.5) (layer "Edge.Cuts") (width 0.05))
   (gr_text "CHECK:position of mounting holes: 86 or 86.5 in y:\nif the position of y is 86 there is the same distance \nbetween mounting hole and top bar and mounting hole\nand capacitor " (at 150.3 66.6) (layer "Dwgs.User")
     (effects (font (size 1.5 1.5) (thickness 0.3)))
   )
+  (dimension (type aligned) (layer "Dwgs.User")
+    (pts (xy 176.15 121.8) (xy 123.65 121.8))
+    (height -14.4)
+    (gr_text "52,5000 mm" (at 149.9 135.05) (layer "Dwgs.User")
+      (effects (font (size 1 1) (thickness 0.15)))
+    )
+    (format (units 3) (units_format 1) (precision 4))
+    (style (thickness 0.1) (arrow_length 1.27) (text_position_mode 0) (extension_height 0.58642) (extension_offset 0.5) keep_text_aligned)
+  )
+  (dimension (type aligned) (layer "Dwgs.User")
+    (pts (xy 176.15 101.8) (xy 176.15 121.8))
+    (height -9.95)
+    (gr_text "20,0000 mm" (at 184.95 111.8 90) (layer "Dwgs.User")
+      (effects (font (size 1 1) (thickness 0.15)))
+    )
+    (format (units 3) (units_format 1) (precision 4))
+    (style (thickness 0.1) (arrow_length 1.27) (text_position_mode 0) (extension_height 0.58642) (extension_offset 0.5) keep_text_aligned)
+  )
+  (dimension (type aligned) (layer "Dwgs.User")
+    (pts (xy 170.6 78.5) (xy 170.6 86))
+    (height 12.4)
+    (gr_text "7,5000 mm" (at 157.05 82.25 90) (layer "Dwgs.User")
+      (effects (font (size 1 1) (thickness 0.15)))
+    )
+    (format (units 3) (units_format 1) (precision 4))
+    (style (thickness 0.1) (arrow_length 1.27) (text_position_mode 0) (extension_height 0.58642) (extension_offset 0.5) keep_text_aligned)
+  )
   (via (at 123.6 108.9) (size 0.8) (drill 0.4) (layers "F.Cu" "B.Cu") (free) (net 1))
