File: dclink.kicad_pcb (KiCad board)
At the start: 2 copper layers, 61.5 x 52.6 mm, 4 parts

Commit message: update vias, fix text on silk, todo: measurement
Parts:
- removed Hello there!: General Kenobi!, LM393:logoleo
Routing:
- net VDC: vias 170 -> 161
- net GND: vias 170 -> 161
Other:
- board text added: "DC-LINK-CAP-EXTENSION JLCJLCJLCJLC"
- board text added: "General Kenobi!"
- board text added: "Hello there!"

Commit message: add measurement
Parts:
- moved   0.25 mm to (170.3, 86.0)
Other:
- board text added: "DC-LINK CAP EXTENSION JLCJLCJLCJLC"
- board text removed: "CHECK:position of mounting holes: 86 or 86.5 in y: if the position of y is 86 there is the same distance between mounting hole and top bar and mounting hole and capacitor"
- board text removed: "DC-LINK-CAP-EXTENSION JLCJLCJLCJLC"

Commit message: minors
Parts:
- moved   0.05 mm to (149.8, 121.3)
